File: kicad/can.sch (KiCad schematic (older format))
At the start: 10 parts, among them J3 8P8C, J4 8P8C, U5 TCAN334

Commit message: Fix errors after first prototype build-up
- Collision of capacitors with MOSFET clamps
- BOOT0 pin tied to GND
- Assignment of a few previously unasigned passives
- Add optional debug serial connector
Parts:
- U5: Manufacturer (none) -> Texas Instruments; PartNumber (none) -> TCAN334
Changed lines of the file:
@@
 Sheet 5 5
 Title "MPPT 2420 RC"
-Date "2020-02-20"
-Rev ""
+Date "2020-05-30"
+Rev "0.1.1"
 Comp "Libre Solar Technologies GmbH"
-Comment1 ""
+Comment1 "Author: Martin Jäger"
 Comment2 ""
 Comment3 ""
@@
 F 2 "LibreSolar:SOIC-8_3.9x4.9mm_Pitch1.27mm" H 3200 2500 50  0001 C CIN
 F 3 "http://www.ti.com/lit/ds/symlink/tcan337.pdf" H 3200 3000 50  0001 C CNN
+F 4 "Texas Instruments" H 3200 3000 50  0001 C CNN "Manufacturer"
+F 5 "TCAN334" H 3200 3000 50  0001 C CNN "PartNumber"
 	1    3200 3000
 	1    0    0    -1

Commit message: Fix some references and part numbers
See issues #3, #5, #7, #8 and #9.
Parts:
- D2, D3: Manufacturer (none) -> ON Semiconductor; PartNumber (none) -> NRVTS260ESFT1G; Remarks (none) -> Alternative: Nexperia PMEG6020ER,115
- J3, J4: Manufacturer (none) -> Amphenol FCI; PartNumber (none) -> 54602-908LF
Changed lines of the file:
@@
 F 2 "LibreSolar:RJ45_8P8C" V 7800 4325 50  0001 C CNN
 F 3 "" V 7800 4325 50  0001 C CNN
+F 4 "Amphenol FCI" H 7800 4300 50  0001 C CNN "Manufacturer"
+F 5 "54602-908LF" H 7800 4300 50  0001 C CNN "PartNumber"
 	1    7800 4300
 	-1   0    0    1
@@
 F 2 "LibreSolar:RJ45_8P8C" V 7800 3025 50  0001 C CNN
 F 3 "" V 7800 3025 50  0001 C CNN
+F 4 "Amphenol FCI" H 7800 3000 50  0001 C CNN "Manufacturer"
+F 5 "54602-908LF" H 7800 3000 50  0001 C CNN "PartNumber"
 	1    7800 3000
 	-1   0    0    1
@@
 F 2 "Diode_SMD:D_SOD-123" H 5500 2400 50  0001 C CNN
 F 3 "" H 5600 2500 50  0001 C CNN
+F 4 "ON Semiconductor" H 5600 2400 50  0001 C CNN "Manufacturer"
+F 5 "NRVTS260ESFT1G" H 5600 2400 50  0001 C CNN "PartNumber"
+F 6 "Alternative: Nexperia PMEG6020ER,115" H 5600 2400 50  0001 C CNN "Remarks"
 	1    5600 2400
 	0    -1   -1   0
@@
 F 2 "Diode_SMD:D_SOD-123" H 6600 5300 50  0001 C CNN
 F 3 "" H 6700 5400 50  0001 C CNN
+F 4 "ON Semiconductor" H 6700 5300 50  0001 C CNN "Manufacturer"
+F 5 "NRVTS260ESFT1G" H 6700 5300 50  0001 C CNN "PartNumber"
+F 6 "Alternative: Nexperia PMEG6020ER,115" H 6700 5300 50  0001 C CNN "Remarks"
 	1    6700 5300
 	0    -1   -1   0

Commit message: Clean up BOM and add build folder for generated files
Parts:
- D2, D3: value D_Schottky -> NRVTS260ESFT1G
- U5: PartNumber TCAN334 -> TCAN334DR
Changed lines of the file:
@@
 F 3 "http://www.ti.com/lit/ds/symlink/tcan337.pdf" H 3200 3000 50  0001 C CNN
 F 4 "Texas Instruments" H 3200 3000 50  0001 C CNN "Manufacturer"
-F 5 "TCAN334" H 3200 3000 50  0001 C CNN "PartNumber"
+F 5 "TCAN334DR" H 3200 3000 50  0001 C CNN "PartNumber"
 	1    3200 3000
 	1    0    0    -1
@@
 P 5600 2400
 F 0 "D2" V 5646 2321 50  0000 R CNN
-F 1 "D_Schottky" V 5555 2321 50  0000 R CNN
+F 1 "NRVTS260ESFT1G" V 5555 2321 50  0000 R CNN
 F 2 "Diode_SMD:D_SOD-123" H 5500 2400 50  0001 C CNN
 F 3 "" H 5600 2500 50  0001 C CNN
@@
 P 6700 5300
 F 0 "D3" V 6746 5221 50  0000 R CNN
-F 1 "D_Schottky" V 6655 5221 50  0000 R CNN
+F 1 "NRVTS260ESFT1G" V 6655 5221 50  0000 R CNN
 F 2 "Diode_SMD:D_SOD-123" H 6600 5300 50  0001 C CNN
 F 3 "" H 6700 5400 50  0001 C CNN
