File: kicad/power-supply.sch (KiCad schematic (older format))
At the start: 25 parts, among them Q9 DMP10H4D2S, T10 MMBT3904, T2 MMBT3904, U4 LMR16006X

Commit message: Fix errors after first prototype build-up
- Collision of capacitors with MOSFET clamps
- BOOT0 pin tied to GND
- Assignment of a few previously unasigned passives
- Add optional debug serial connector
Parts:
- C41: value 4.7µF -> 2.2µF; Manufacturer Wurth Electronics -> (none); PartNumber 885012107018 -> (none)
- R60: value 12k -> 33k; PartNumber RC0805FR-0712KL -> RC0805FR-0733KL
- R64, R65, R66: value 12k -> 10k; PartNumber RC0805FR-0712KL -> RC0805FR-0710KL
Changed lines of the file:
@@
 Sheet 3 5
 Title "MPPT 2420 RC"
-Date "2020-02-20"
-Rev "0.1"
+Date "2020-05-30"
+Rev "0.1.1"
 Comp "Libre Solar Technologies GmbH"
 Comment1 "Author: Martin Jäger"
@@
 AR Path="/58C18D5C/5DA192E6" Ref="R64"  Part="1"
 F 0 "R64" V 4475 5500 50  0000 C CNN
-F 1 "12k" V 4300 5500 50  0000 C CNN
+F 1 "10k" V 4300 5500 50  0000 C CNN
 F 2 "LibreSolar:R_0603_1608" H 4400 5500 50  0001 C CNN
 F 3 "" H 4400 5500 50  0001 C CNN
 F 4 "Yageo" H 4400 5500 50  0001 C CNN "Manufacturer"
-F 5 "RC0805FR-0712KL" H 4400 5500 50  0001 C CNN "PartNumber"
+F 5 "RC0805FR-0710KL" H 4400 5500 50  0001 C CNN "PartNumber"
 	1    4400 5500
 	-1   0    0    1
@@
 AR Path="/58C18D5C/5DA192F5" Ref="C41"  Part="1"
 F 0 "C41" H 5225 5775 50  0000 L CNN
-F 1 "4.7µF" H 5225 5625 50  0000 L CNN
+F 1 "2.2µF" H 5225 5625 50  0000 L CNN
 F 2 "LibreSolar:C_0603_1608" H 5200 5500 50  0001 C CNN
 F 3 "" H 5225 5775 50  0000 C CNN
-F 4 "Wurth Electronics" H -2800 2950 50  0001 C CNN "Manufacturer"
-F 5 "885012107018" H -2800 2950 50  0001 C CNN "PartNumber"
-F 6 "25V, X5R" H -600 400 60  0001 C CNN "Remarks"
+F 4 "25V, X5R" H -600 400 60  0001 C CNN "Remarks"
 	1    5200 5700
 	1    0    0    -1
@@
 AR Path="/58C18D5C/5E0849FF" Ref="R66"  Part="1"
 F 0 "R66" V 2675 3200 50  0000 C CNN
-F 1 "12k" V 2500 3200 50  0000 C CNN
+F 1 "10k" V 2500 3200 50  0000 C CNN
 F 2 "LibreSolar:R_0603_1608" H 2600 3200 50  0001 C CNN
 F 3 "" H 2600 3200 50  0001 C CNN
 F 4 "Yageo" H 2600 3200 50  0001 C CNN "Manufacturer"
-F 5 "RC0805FR-0712KL" H 2600 3200 50  0001 C CNN "PartNumber"
+F 5 "RC0805FR-0710KL" H 2600 3200 50  0001 C CNN "PartNumber"
 	1    2600 3200
 	-1   0    0    1
@@
 AR Path="/58C18D5C/5E0855A8" Ref="R60"  Part="1"
 F 0 "R60" V 1775 3200 50  0000 C CNN
-F 1 "12k" V 1600 3200 50  0000 C CNN
+F 1 "33k" V 1600 3200 50  0000 C CNN
 F 2 "LibreSolar:R_0603_1608" H 1700 3200 50  0001 C CNN
 F 3 "" H 1700 3200 50  0001 C CNN
 F 4 "Yageo" H 1700 3200 50  0001 C CNN "Manufacturer"
-F 5 "RC0805FR-0712KL" H 1700 3200 50  0001 C CNN "PartNumber"
+F 5 "RC0805FR-0733KL" H 1700 3200 50  0001 C CNN "PartNumber"
 	1    1700 3200
 	-1   0    0    1
@@
 AR Path="/58C18D5C/5E0B3D6C" Ref="R65"  Part="1"
 F 0 "R65" V 2075 2600 50  0000 C CNN
-F 1 "12k" V 1900 2600 50  0000 C CNN
+F 1 "10k" V 1900 2600 50  0000 C CNN
 F 2 "LibreSolar:R_0603_1608" H 2000 2600 50  0001 C CNN
 F 3 "" H 2000 2600 50  0001 C CNN
 F 4 "Yageo" H 2000 2600 50  0001 C CNN "Manufacturer"
-F 5 "RC0805FR-0712KL" H 2000 2600 50  0001 C CNN "PartNumber"
+F 5 "RC0805FR-0710KL" H 2000 2600 50  0001 C CNN "PartNumber"
 	1    2000 2600
 	-1   0    0    1

Commit message: Fix some references and part numbers
See issues #3, #5, #7, #8 and #9.
Parts:
- C41: Manufacturer (none) -> Murata; PartNumber (none) -> GRM188R61E225KA12D
- R60: PartNumber RC0805FR-0733KL -> RC0603FR-0733KL
- R64, R65, R66: PartNumber RC0805FR-0710KL -> RC0603FR-0710KL
Changed lines of the file:
@@
 F 3 "" H 4400 5500 50  0001 C CNN
 F 4 "Yageo" H 4400 5500 50  0001 C CNN "Manufacturer"
-F 5 "RC0805FR-0710KL" H 4400 5500 50  0001 C CNN "PartNumber"
+F 5 "RC0603FR-0710KL" H 4400 5500 50  0001 C CNN "PartNumber"
 	1    4400 5500
 	-1   0    0    1
@@
 F 3 "" H 5225 5775 50  0000 C CNN
 F 4 "25V, X5R" H -600 400 60  0001 C CNN "Remarks"
+F 5 "Murata" H 5200 5700 50  0001 C CNN "Manufacturer"
+F 6 "GRM188R61E225KA12D" H 5200 5700 50  0001 C CNN "PartNumber"
 	1    5200 5700
 	1    0    0    -1
@@
 F 3 "" H 2600 3200 50  0001 C CNN
 F 4 "Yageo" H 2600 3200 50  0001 C CNN "Manufacturer"
-F 5 "RC0805FR-0710KL" H 2600 3200 50  0001 C CNN "PartNumber"
+F 5 "RC0603FR-0710KL" H 2600 3200 50  0001 C CNN "PartNumber"
 	1    2600 3200
 	-1   0    0    1
@@
 F 3 "" H 1700 3200 50  0001 C CNN
 F 4 "Yageo" H 1700 3200 50  0001 C CNN "Manufacturer"
-F 5 "RC0805FR-0733KL" H 1700 3200 50  0001 C CNN "PartNumber"
+F 5 "RC0603FR-0733KL" H 1700 3200 50  0001 C CNN "PartNumber"
 	1    1700 3200
 	-1   0    0    1
@@
 F 3 "" H 2000 2600 50  0001 C CNN
 F 4 "Yageo" H 2000 2600 50  0001 C CNN "Manufacturer"
-F 5 "RC0805FR-0710KL" H 2000 2600 50  0001 C CNN "PartNumber"
+F 5 "RC0603FR-0710KL" H 2000 2600 50  0001 C CNN "PartNumber"
 	1    2000 2600
 	-1   0    0    1

Commit message: Clean up BOM and add build folder for generated files
Parts:
- D1: Alternative DFLS160-7 -> (none); Remarks (none) -> Alternative: DFLS160-7
- L3: Alternative Bourns SRR6045TA-470Y -> (none); Remarks (none) -> Alternative: Bourns SRR6045TA-470Y
Changed lines of the file:
@@
 F 4 "Diodes Inc." H 2700 100 50  0001 C CNN "Manufacturer"
 F 5 "SS16FP" H 2700 100 50  0001 C CNN "PartNumber"
-F 6 "DFLS160-7" H 1300 -100 60  0001 C CNN "Alternative"
+F 6 "" H 1300 -100 60  0001 C CNN "Alternative"
+F 7 "Alternative: DFLS160-7" H 7400 2700 50  0001 C CNN "Remarks"
 	1    7400 2700
 	0    -1   1    0
@@
 F 4 "Tayo Yuden" H 7950 2500 60  0001 C CNN "Manufacturer"
 F 5 "NR6045T470M" H 7950 2500 60  0001 C CNN "PartNumber"
-F 6 "Bourns SRR6045TA-470Y" H 7950 2500 60  0001 C CNN "Alternative"
+F 6 "" H 7950 2500 60  0001 C CNN "Alternative"
+F 7 "Alternative: Bourns SRR6045TA-470Y" H 7950 2500 50  0001 C CNN "Remarks"
 	1    7950 2500
 	0    -1   -1   0
